File: CustomKeyboardKiCAD/LEDs.kicad_sch (KiCad schematic)
At the start: 99 parts, among them U8 74AHC1G125

Commit message: schematic is generally complete
Parts:
- added F1: 2A, 2amp_polyfuse:FUSE_1812L200_LTF, symbol Device:Polyfuse
- C29: value 100uF -> 220uF; footprint (none) -> GRM31CD80J107MEA8L:GRM31x
- C30: footprint (none) -> C0603C104K5RACTU:CAPC1608X90
- D100, D101, D102, D103, D104, D105, D106, D107, D108, D109, D110, D111, D112, D113, D114, D115, D116, D117, D118, D119, D120, D121, D122, D123, D124, D125, D126, D127, D128, D129, D130, D131, D132, D133, D134, D135, D136, D137, D138, D139, D140, D141, D142, D143, D144, D145, D146, D147, D148, D149, D150, D151, D152, D153, D154, D155, D156, D157, D158, D159, D160, D161, D162, D163, D164, D165, D166, D167, D168, D169, D17, D170, D171, D172, D173, D174, D175, D176, D177, D178, D179, D18, D180, D181, D182, D183, D184, D185, D93, D94, D95, D96, D97, D98, D99: footprint LED_SMD:LED_WS2812B_PLCC4_5.0x5.0mm_P3.2mm -> ADDRESS LED:COM-16347_SPK
- R10: footprint (none) -> RC0603JR-07330RL:RESC1608X55N
Connections:
- net VBUS: now also F1.2; no longer C29.2, D100.1 (VDD), D101.1 (VDD), D102.1 (VDD), D103.1 (VDD), D104.1 (VDD), D105.1 (VDD), D106.1 (VDD), D107.1 (VDD), D108.1 (VDD), D109.1 (VDD), D110.1 (VDD), D111.1 (VDD), D112.1 (VDD), D113.1 (VDD), D114.1 (VDD), D115.1 (VDD), D116.1 (VDD), D117.1 (VDD), D118.1 (VDD), D119.1 (VDD), D120.1 (VDD), D121.1 (VDD), D122.1 (VDD), D123.1 (VDD), D124.1 (VDD), D125.1 (VDD), D126.1 (VDD), D127.1 (VDD), D128.1 (VDD), D129.1 (VDD), D130.1 (VDD), D131.1 (VDD), D132.1 (VDD), D133.1 (VDD), D134.1 (VDD), D135.1 (VDD), D136.1 (VDD), D137.1 (VDD), D138.1 (VDD), D139.1 (VDD), D140.1 (VDD), D141.1 (VDD), D142.1 (VDD), D143.1 (VDD), D144.1 (VDD), D145.1 (VDD), D146.1 (VDD), D147.1 (VDD), D148.1 (VDD), D149.1 (VDD), D150.1 (VDD), D151.1 (VDD), D152.1 (VDD), D153.1 (VDD), D154.1 (VDD), D155.1 (VDD), D156.1 (VDD), D157.1 (VDD), D158.1 (VDD), D159.1 (VDD), D160.1 (VDD), D161.1 (VDD), D162.1 (VDD), D163.1 (VDD), D164.1 (VDD), D165.1 (VDD), D166.1 (VDD), D167.1 (VDD), D168.1 (VDD), D169.1 (VDD), D17.1 (VDD), D170.1 (VDD), D171.1 (VDD), D172.1 (VDD), D173.1 (VDD), D174.1 (VDD), D175.1 (VDD), D176.1 (VDD), D177.1 (VDD), D178.1 (VDD), D179.1 (VDD), D18.1 (VDD), D180.1 (VDD), D181.1 (VDD), D182.1 (VDD), D183.1 (VDD), D184.1 (VDD), D185.1 (VDD), D93.1 (VDD), D94.1 (VDD), D95.1 (VDD), D96.1 (VDD), D97.1 (VDD), D98.1 (VDD), D99.1 (VDD)
- new net: C29.2, D100.1 (VDD), D101.1 (VDD), D102.1 (VDD), D103.1 (VDD), D104.1 (VDD), D105.1 (VDD), D106.1 (VDD), D107.1 (VDD), D108.1 (VDD), D109.1 (VDD), D110.1 (VDD), D111.1 (VDD), D112.1 (VDD), D113.1 (VDD), D114.1 (VDD), D115.1 (VDD), D116.1 (VDD), D117.1 (VDD), D118.1 (VDD), D119.1 (VDD), D120.1 (VDD), D121.1 (VDD), D122.1 (VDD), D123.1 (VDD), D124.1 (VDD), D125.1 (VDD), D126.1 (VDD), D127.1 (VDD), D128.1 (VDD), D129.1 (VDD), D130.1 (VDD), D131.1 (VDD), D132.1 (VDD), D133.1 (VDD), D134.1 (VDD), D135.1 (VDD), D136.1 (VDD), D137.1 (VDD), D138.1 (VDD), D139.1 (VDD), D140.1 (VDD), D141.1 (VDD), D142.1 (VDD), D143.1 (VDD), D144.1 (VDD), D145.1 (VDD), D146.1 (VDD), D147.1 (VDD), D148.1 (VDD), D149.1 (VDD), D150.1 (VDD), D151.1 (VDD), D152.1 (VDD), D153.1 (VDD), D154.1 (VDD), D155.1 (VDD), D156.1 (VDD), D157.1 (VDD), D158.1 (VDD), D159.1 (VDD), D160.1 (VDD), D161.1 (VDD), D162.1 (VDD), D163.1 (VDD), D164.1 (VDD), D165.1 (VDD), D166.1 (VDD), D167.1 (VDD), D168.1 (VDD), D169.1 (VDD), D17.1 (VDD), D170.1 (VDD), D171.1 (VDD), D172.1 (VDD), D173.1 (VDD), D174.1 (VDD), D175.1 (VDD), D176.1 (VDD), D177.1 (VDD), D178.1 (VDD), D179.1 (VDD), D18.1 (VDD), D180.1 (VDD), D181.1 (VDD), D182.1 (VDD), D183.1 (VDD), D184.1 (VDD), D185.1 (VDD), D93.1 (VDD), D94.1 (VDD), D95.1 (VDD), D96.1 (VDD), D97.1 (VDD), D98.1 (VDD), D99.1 (VDD), F1.1
Other:
- moved on the sheet: C29, C30, D100, D101, D102, D103, D104, D105, D106, D107, D108, D109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

Commit message: major progress on pcb, schematic complete
Parts:
- removed C29: 220uF, GRM31CD80J107MEA8L:GRM31x, symbol Device:C
- removed D100, D101, D102, D103, D104, D105, D106, D107, D108, D109, D110, D111, D112, D113, D114, D115, D116, D117, D118, D119, D120, D121, D122, D123, D124, D125, D126, D127, D128, D129, D130, D131, D132, D133, D134, D135, D136, D137, D138, D139, D140, D141, D142, D143, D144, D145, D146, D147, D148, D149, D150, D151, D152, D153, D154, D155, D156, D157, D158, D159, D160, D161, D162, D163, D164, D165, D166, D167, D168, D169, D17, D170, D171, D172, D173, D174, D175, D176, D177, D178, D179, D18, D180, D181, D182, D183, D184, D185, D93, D94, D95, D96, D97, D98, D99: WS2812B, ADDRESS LED:COM-16347_SPK, symbol LED:WS2812B
- removed F1: 2A, 2amp_polyfuse:FUSE_1812L200_LTF, symbol Device:Polyfuse
- added C31: 220uF, 220uF:GRM31x, symbol Device:C
- added F2: 2A, 2amp_polyfuse:FUSE_1812L200_LTF, symbol Device:Polyfuse
- added LED1, LED10, LED100, LED11, LED12, LED13, LED14, LED15, LED16, LED17, LED18, LED19, LED2, LED20, LED21, LED22, LED23, LED25, LED26, LED27, LED28, LED29, LED3, LED30, LED31, LED32, LED33, LED34, LED35, LED36, LED37, LED38, LED39, LED4, LED40, LED41, LED42, LED43, LED44, LED45, LED46, LED47, LED48, LED49, LED5, LED50, LED51, LED52, LED53, LED54, LED55, LED56, LED57, LED58, LED59, LED6, LED60, LED61, LED62, LED63, LED64, LED65, LED66, LED67, LED68, LED69, LED7, LED70, LED71, LED72, LED73, LED74, LED75, LED76, LED77, LED78, LED79, LED8, LED80, LED81, LED82, LED83, LED84, LED85, LED86, LED87, LED88, LED89, LED9, LED90, LED91, LED92, LED93, LED94, LED95, LED96, LED97, LED98, LED99: ~, ai03:LED-SMD_4P-L3.2-W2.8-LS5.9_SK6812MINI-E, symbol SK6812MINI-E:SK6812MINI-E_C5149201
- U8: footprint 74HC595D:SOP127P600X175-16N -> SN74AHC1G125DCKR:SOT65P210X110-5N
Connections:
- net D_in: now also LED1.2 (DIN)
- net GND: now also C31.1, LED1.1 (GND), LED10.1 (GND), LED100.1 (GND), LED11.1 (GND), LED12.1 (GND), LED13.1 (GND), LED14.1 (GND), LED15.1 (GND), LED16.1 (GND), LED17.1 (GND), LED18.1 (GND), LED19.1 (GND), LED2.1 (GND), LED20.1 (GND), LED21.1 (GND), LED22.1 (GND), LED23.1 (GND), LED25.1 (GND), LED26.1 (GND), LED27.1 (GND), LED28.1 (GND), LED29.1 (GND), LED3.1 (GND), LED30.1 (GND), LED31.1 (GND), LED32.1 (GND), LED33.1 (GND), LED34.1 (GND), LED35.1 (GND), LED36.1 (GND), LED37.1 (GND), LED38.1 (GND), LED39.1 (GND), LED4.1 (GND), LED40.1 (GND), LED41.1 (GND), LED42.1 (GND), LED43.1 (GND), LED44.1 (GND), LED45.1 (GND), LED46.1 (GND), LED47.1 (GND), LED48.1 (GND), LED49.1 (GND), LED5.1 (GND), LED50.1 (GND), LED51.1 (GND), LED52.1 (GND), LED53.1 (GND), LED54.1 (GND), LED55.1 (GND), LED56.1 (GND), LED57.1 (GND), LED58.1 (GND), LED59.1 (GND), LED6.1 (GND), LED60.1 (GND), LED61.1 (GND), LED62.1 (GND), LED63.1 (GND), LED64.1 (GND), LED65.1 (GND), LED66.1 (GND), LED67.1 (GND), LED68.1 (GND), LED69.1 (GND), LED7.1 (GND), LED70.1 (GND), LED71.1 (GND), LED72.1 (GND), LED73.1 (GND), LED74.1 (GND), LED75.1 (GND), LED76.1 (GND), LED77.1 (GND), LED78.1 (GND), LED79.1 (GND), LED8.1 (GND), LED80.1 (GND), LED81.1 (GND), LED82.1 (GND), LED83.1 (GND), LED84.1 (GND), LED85.1 (GND), LED86.1 (GND), LED87.1 (GND), LED88.1 (GND), LED89.1 (GND), LED9.1 (GND), LED90.1 (GND), LED91.1 (GND), LED92.1 (GND), LED93.1 (GND), LED94.1 (GND), LED95.1 (GND), LED96.1 (GND), LED97.1 (GND), LED98.1 (GND), LED99.1 (GND)
- net VBUS: now also F2.2
- new net: LED22.4 (DOUT), LED23.2 (DIN)
- new net: LED23.4 (DOUT), LED25.2 (DIN)
- new net: LED51.4 (DOUT), LED52.2 (DIN)
- new net: LED52.4 (DOUT), LED53.2 (DIN)
- new net: LED2.4 (DOUT), LED3.2 (DIN)
- new net: LED3.4 (DOUT), LED4.2 (DIN)
- new net: LED88.4 (DOUT), LED89.2 (DIN)
- new net: LED89.4 (DOUT), LED90.2 (DIN)
- new net: LED66.4 (DOUT), LED67.2 (DIN)
- new net: LED67.4 (DOUT), LED68.2 (DIN)
- new net: LED44.4 (DOUT), LED45.2 (DIN)
- new net: LED45.4 (DOUT), LED46.2 (DIN)
- new net: LED55.4 (DOUT), LED56.2 (DIN)
- new net: LED56.4 (DOUT), LED57.2 (DIN)
- new net: LED4.4 (DOUT), LED5.2 (DIN)
- new net: LED32.4 (DOUT), LED33.2 (DIN)
- new net: LED33.4 (DOUT), LED34.2 (DIN)
- new net: LED76.4 (DOUT), LED77.2 (DIN)
- new net: LED77.4 (DOUT), LED78.2 (DIN)
- new net: LED87.4 (DOUT), LED88.2 (DIN)
- new net: LED48.4 (DOUT), LED49.2 (DIN)
- new net: LED49.4 (DOUT), LED50.2 (DIN)
- new net: LED80.4 (DOUT), LED81.2 (DIN)
- new net: LED81.4 (DOUT), LED82.2 (DIN)
- new net: LED18.4 (DOUT), LED19.2 (DIN)
- new net: LED19.4 (DOUT), LED20.2 (DIN)
- new net: LED14.4 (DOUT), LED15.2 (DIN)
- new net: LED15.4 (DOUT), LED16.2 (DIN)
- new net: LED30.4 (DOUT), LED31.2 (DIN)
- new net: LED31.4 (DOUT), LED32.2 (DIN)
- new net: LED97.4 (DOUT), LED98.2 (DIN)
- new net: LED98.4 (DOUT), LED99.2 (DIN)
- new net: LED39.4 (DOUT), LED40.2 (DIN)
- new net: LED40.4 (DOUT), LED41.2 (DIN)
- new net: LED47.4 (DOUT), LED48.2 (DIN)
- new net: LED94.4 (DOUT), LED95.2 (DIN)
- new net: LED95.4 (DOUT), LED96.2 (DIN)
- new net: LED96.4 (DOUT), LED97.2 (DIN)
- new net: LED93.4 (DOUT), LED94.2 (DIN)
- new net: LED58.4 (DOUT), LED59.2 (DIN)
- new net: LED59.4 (DOUT), LED60.2 (DIN)
- new net: LED60.4 (DOUT), LED61.2 (DIN)
- new net: LED75.4 (DOUT), LED76.2 (DIN)
- new net: LED62.4 (DOUT), LED63.2 (DIN)
- new net: LED63.4 (DOUT), LED64.2 (DIN)
- new net: LED12.4 (DOUT), LED13.2 (DIN)
- new net: LED13.4 (DOUT), LED14.2 (DIN)
- new net: LED16.4 (DOUT), LED17.2 (DIN)
- new net: LED17.4 (DOUT), LED18.2 (DIN)
- new net: LED27.4 (DOUT), LED28.2 (DIN)
- new net: LED28.4 (DOUT), LED29.2 (DIN)
- new net: LED71.4 (DOUT), LED72.2 (DIN)
- new net: LED72.4 (DOUT), LED73.2 (DIN)
- new net: LED21.4 (DOUT), LED22.2 (DIN)
- new net: LED90.4 (DOUT), LED91.2 (DIN)
- new net: LED91.4 (DOUT), LED92.2 (DIN)
- new net: LED35.4 (DOUT), LED36.2 (DIN)
- new net: LED36.4 (DOUT), LED37.2 (DIN)
- new net: LED54.4 (DOUT), LED55.2 (DIN)
- new net: LED85.4 (DOUT), LED86.2 (DIN)
- new net: LED86.4 (DOUT), LED87.2 (DIN)
- new net: LED37.4 (DOUT), LED38.2 (DIN)
- new net: LED38.4 (DOUT), LED39.2 (DIN)
- new net: LED41.4 (DOUT), LED42.2 (DIN)
- new net: LED42.4 (DOUT), LED43.2 (DIN)
- new net: LED10.2 (DIN), LED9.4 (DOUT)
- new net: LED10.4 (DOUT), LED11.2 (DIN)
- new net: LED5.4 (DOUT), LED6.2 (DIN)
- new net: LED6.4 (DOUT), LED7.2 (DIN)
- new net: LED100.2 (DIN), LED99.4 (DOUT)
- new net: LED20.4 (DOUT), LED21.2 (DIN)
- new net: LED43.4 (DOUT), LED44.2 (DIN)
- new net: LED53.4 (DOUT), LED54.2 (DIN)
- new net: LED73.4 (DOUT), LED74.2 (DIN)
- new net: LED74.4 (DOUT), LED75.2 (DIN)
- new net: LED11.4 (DOUT), LED12.2 (DIN)
- new net: LED92.4 (DOUT), LED93.2 (DIN)
- new net: LED68.4 (DOUT), LED69.2 (DIN)
- new net: LED69.4 (DOUT), LED70.2 (DIN)
- new net: LED34.4 (DOUT), LED35.2 (DIN)
- new net: LED29.4 (DOUT), LED30.2 (DIN)
- new net: LED46.4 (DOUT), LED47.2 (DIN)
- new net: LED64.4 (DOUT), LED65.2 (DIN)
- new net: LED65.4 (DOUT), LED66.2 (DIN)
- new net: LED50.4 (DOUT), LED51.2 (DIN)
- new net: LED25.4 (DOUT), LED26.2 (DIN)
- new net: LED7.4 (DOUT), LED8.2 (DIN)
- new net: LED8.4 (DOUT), LED9.2 (DIN)
- new net: LED61.4 (DOUT), LED62.2 (DIN)
- new net: LED57.4 (DOUT), LED58.2 (DIN)
- new net: LED82.4 (DOUT), LED83.2 (DIN)
- new net: LED83.4 (DOUT), LED84.2 (DIN)
- new net: LED70.4 (DOUT), LED71.2 (DIN)
- new net: LED1.4 (DOUT), LED2.2 (DIN)
- new net: LED84.4 (DOUT), LED85.2 (DIN)
- new net: LED78.4 (DOUT), LED79.2 (DIN)
- new net: LED26.4 (DOUT), LED27.2 (DIN)
- new net: LED79.4 (DOUT), LED80.2 (DIN)
- new net LED5V_NET: C31.2, F2.1, LED1.3 (VDD), LED10.3 (VDD), LED100.3 (VDD), LED11.3 (VDD), LED12.3 (VDD), LED13.3 (VDD), LED14.3 (VDD), LED15.3 (VDD), LED16.3 (VDD), LED17.3 (VDD), LED18.3 (VDD), LED19.3 (VDD), LED2.3 (VDD), LED20.3 (VDD), LED21.3 (VDD), LED22.3 (VDD), LED23.3 (VDD), LED25.3 (VDD), LED26.3 (VDD), LED27.3 (VDD), LED28.3 (VDD), LED29.3 (VDD), LED3.3 (VDD), LED30.3 (VDD), LED31.3 (VDD), LED32.3 (VDD), LED33.3 (VDD), LED34.3 (VDD), LED35.3 (VDD), LED36.3 (VDD), LED37.3 (VDD), LED38.3 (VDD), LED39.3 (VDD), LED4.3 (VDD), LED40.3 (VDD), LED41.3 (VDD), LED42.3 (VDD), LED43.3 (VDD), LED44.3 (VDD), LED45.3 (VDD), LED46.3 (VDD), LED47.3 (VDD), LED48.3 (VDD), LED49.3 (VDD), LED5.3 (VDD), LED50.3 (VDD), LED51.3 (VDD), LED52.3 (VDD), LED53.3 (VDD), LED54.3 (VDD), LED55.3 (VDD), LED56.3 (VDD), LED57.3 (VDD), LED58.3 (VDD), LED59.3 (VDD), LED6.3 (VDD), LED60.3 (VDD), LED61.3 (VDD), LED62.3 (VDD), LED63.3 (VDD), LED64.3 (VDD), LED65.3 (VDD), LED66.3 (VDD), LED67.3 (VDD), LED68.3 (VDD), LED69.3 (VDD), LED7.3 (VDD), LED70.3 (VDD), LED71.3 (VDD), LED72.3 (VDD), LED73.3 (VDD), LED74.3 (VDD), LED75.3 (VDD), LED76.3 (VDD), LED77.3 (VDD), LED78.3 (VDD), LED79.3 (VDD), LED8.3 (VDD), LED80.3 (VDD), LED81.3 (VDD), LED82.3 (VDD), LED83.3 (VDD), LED84.3 (VDD), LED85.3 (VDD), LED86.3 (VDD), LED87.3 (VDD), LED88.3 (VDD), LED89.3 (VDD), LED9.3 (VDD), LED90.3 (VDD), LED91.3 (VDD), LED92.3 (VDD), LED93.3 (VDD), LED94.3 (VDD), LED95.3 (VDD), LED96.3 (VDD), LED97.3 (VDD), LED98.3 (VDD), LED99.3 (VDD)

Commit message: more progress on pcb
Parts:
- removed LED55: ~, ai03:LED-SMD_4P-L3.2-W2.8-LS5.9_SK6812MINI-E, symbol SK6812MINI-E:SK6812MINI-E_C5149201
Connections:
- net at LED56.2 (DIN): now also LED54.4 (DOUT)
Changed lines of the file:
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@@
 	(wire
 		(pts
-			(xy 949.96 219.71) (xy 955.04 219.71)
-		)
-		(stroke
-			(width 0)
-			(type default)
-		)
-	)
-	(wire
-		(pts
 			(xy 435.61 219.71) (xy 440.69 219.71)
 		)
@@
 	(wire
 		(pts
-			(xy 915.67 219.71) (xy 920.75 219.71)
+			(xy 915.67 219.71) (xy 955.04 219.71)
 		)
 		(stroke
@@
 	(wire
 		(pts
-			(xy 941.07 217.17) (xy 949.96 217.17)
-		)
-		(stroke
-			(width 0)
-			(type default)
-		)
-	)
-	(wire
-		(pts
 			(xy 906.78 217.17) (xy 915.67 217.17)
 		)
@@
 	(wire
 		(pts
-			(xy 949.96 217.17) (xy 949.96 219.71)
-		)
-		(stroke
-			(width 0)
-			(type default)
-		)
-	)
-	(wire
-		(pts
 			(xy 1018.54 180.34) (xy 1018.54 182.88)
 		)
@@
 	(global_label "LED5V_NET"
 		(shape input)
-		(at 941.07 219.71 270)
-		(fields_autoplaced yes)
-		(effects
-			(font
-				(size 1.27 1.27)
-			)
-			(justify right)
-		)
-		(property "Intersheetrefs" "${INTERSHEET_REFS}"
-			(at 941.07 232.8551 90)
-			(effects
-				(font
-					(size 1.27 1.27)
-				)
-				(justify right)
-				(hide yes)
-			)
-		)
-	)
-	(global_label "LED5V_NET"
-		(shape input)
 		(at 1045.21 246.38 270)
 		(fields_autoplaced yes)
@@
 	)
 	(symbol
-		(lib_id "SK6812MINI-E:SK6812MINI-E_C5149201")
-		(at 930.91 218.44 0)
-		(unit 1)
-		(exclude_from_sim no)
-		(in_bom yes)
-		(on_board yes)
-		(dnp no)
-		(fields_autoplaced yes)
-		(property "Reference" "LED55"
-			(at 930.91 209.55 0)
-			(effects
-				(font
-					(size 1.27 1.27)
-				)
-			)
-		)
-		(property "Value" "~"
-			(at 930.91 212.09 0)
-			(effects
-				(font
-					(size 1.27 1.27)
-				)
-			)
-		)
-		(property "Footprint" "ai03:LED-SMD_4P-L3.2-W2.8-LS5.9_SK6812MINI-E"
-			(at 930.91 218.44 0)
-			(effects
-				(font
-					(size 1.27 1.27)
-				)
-				(hide yes)
-			)
-		)
-		(property "Datasheet" "https://item.szlcsc.com/datasheet/SK6812MINI-E/5773397.html"
-			(at 930.91 218.44 0)
-			(effects
-				(font
-					(size 1.27 1.27)
-				)
-				(hide yes)
-			)
-		)
-		(property "Description" ""
-			(at 930.91 218.44 0)
-			(effects
-				(font
-					(size 1.27 1.27)
-				)
-				(hide yes)
-			)
-		)
-		(property "Manufacturer Part" "SK6812MINI-E"
-			(at 930.91 218.44 0)
-			(effects
-				(font
-					(size 1.27 1.27)
-				)
-				(hide yes)
-			)
-		)
-		(property "Manufacturer" "欧思科光电"
-			(at 930.91 218.44 0)
-			(effects
-				(font
-					(size 1.27 1.27)
-				)
-				(hide yes)
-			)
-		)
-		(property "Supplier Part" "C5149201"
-			(at 930.91 218.44 0)
-			(effects
-				(font
-					(size 1.27 1.27)
-				)
-				(hide yes)
-			)
-		)
-		(property "Supplier" "LCSC"
-			(at 930.91 218.44 0)
-			(effects
-				(font
-					(size 1.27 1.27)
-				)
-				(hide yes)
-			)
-		)
-		(property "LCSC Part Name" "SK6812MINI-E"
-			(at 930.91 218.44 0)
-			(effects
-				(font
-					(size 1.27 1.27)
-				)
-				(hide yes)
-			)
-		)
-		(pin "2"
-		)
-		(pin "1"
-		)
-		(pin "4"
-		)
-		(pin "3"
-		)
-		(instances
-			(project "CustomKeyboardKiCAD"
-				(path "/aaa1400c-18c9-4b83-ab7e-c530ca104a6d/b1111ac9-608b-4dfe-b586-313897de2924"
-					(reference "LED55")
-					(unit 1)
-				)
-			)
-		)
-	)
-	(symbol
 		(lib_id "power:GND")
 		(at 337.82 180.34 270)
@@
 					(unit 1)
 				)
-			)
-		)
-	)
-	(symbol
-		(lib_id "power:GND")
-		(at 920.75 217.17 270)
-		(unit 1)
-		(exclude_from_sim no)
-		(in_bom yes)
-		(on_board yes)
-		(dnp no)
-		(fields_autoplaced yes)
-		(property "Reference" "#PWR0111"
-			(at 914.4 217.17 0)
-			(effects
-				(font
-					(size 1.27 1.27)
-				)
-				(hide yes)
-			)
-		)
-		(property "Value" "GND"
-			(at 919.48 213.36 90)
-			(effects
-				(font
-					(size 1.27 1.27)
-				)
-			)
-		)
-		(property "Footprint" ""
-			(at 920.75 217.17 0)
-			(effects
-				(font
-					(size 1.27 1.27)
-				)
-				(hide yes)
-			)
-		)
-		(property "Datasheet" ""
-			(at 920.75 217.17 0)
-			(effects
-				(font
-					(size 1.27 1.27)
-				)
-				(hide yes)
-			)
-		)
-		(property "Description" "Power symbol creates a global label with name \"GND\" , ground"
-			(at 920.75 217.17 0)
-			(effects
-				(font
-					(size 1.27 1.27)
-				)
-				(hide yes)
-			)
-		)
-		(pin "1"
-		)
-		(instances
-			(project "CustomKeyboardKiCAD"
-				(path "/aaa1400c-18c9-4b83-ab7e-c530ca104a6d/b1111ac9-608b-4dfe-b586-313897de2924"
-					(reference "#PWR0111")
-					(unit 1)
-				)

Commit message: pcb complete
Connections:
- net VBUS renamed V_5VOUTUSB
